Commit message: Comments added to URDF file
comments added to the omni.urdf.xacro file in omni_description for clarity.

Next update: visual compass package.

File: omni_description/urdf/omni.urdf.xacro (robot description, xacro)
@@ -1,4 +1,5 @@
 <?xml version="1.0"?>
 <robot xmlns:xacro="http://www.ros.org/wiki/xacro" name="omni">
+<!--ROS Gazebo plugin-->
 <gazebo>
   <plugin name="gazebo_ros_control" filename="libgazebo_ros_control.so">
@@ -6,4 +7,5 @@
   </plugin>
 </gazebo>
+<!--xacro constants used for robot dimensions-->
 <xacro:property name="wb_w" value="0.18"/>
 <xacro:property name="wb_h" value="0.005"/>
@@ -14,5 +16,6 @@
 <xacro:property name="ct_d" value="${wb_d/1.51}"/>
 <xacro:property name="ct_m" value="${((ct_w*ct_d)/(wb_w*wb_d))*wb_m}"/>
-<xacro:property name="camera_link" value="0.05" /> <!-- Size of square 'camera' box -->
+<!-- Size of square 'camera' box -->
+<xacro:property name="camera_link" value="0.05" />
 <xacro:property name="p_r" value="0.0025"/>
 <xacro:property name="p_l" value="0.0515"/>
@@ -23,4 +26,5 @@
 <xacro:property name="b_r" value="0.024"/>
 <xacro:property name="b_m" value="0.60"/>
+<!--macros used to define inertia and geometry tags-->
 <xacro:macro name="wb_inertial" params="mass depth width height">
   <inertial>
@@ -83,4 +87,5 @@
     </inertial>
 </xacro:macro>
+  <!-- link definitions-->
   <link name = "wheel_base">
     <visual>
@@ -90,4 +95,5 @@
       <xacro:wb_dim depth="${wb_d}" width="${wb_w}" height="${wb_h}"/>
     </collision>
+    <!--depth, width and height parameters are squared before being passed in, to simplify inertia calculations-->
     <xacro:wb_inertial mass="${wb_m}" depth="${wb_d*wb_d}" width="${wb_w*wb_w}" height="${wb_h*wb_h}"/>
   </link>
@@ -99,4 +105,5 @@
       <xacro:wb_dim depth="${ct_d}" width="${ct_w}" height="${ct_h}"/>
     </collision>
+    <!--depth, width and height parameters are squared before being passed in, to simplify inertia calculations-->
     <xacro:wb_inertial mass="${wb_m}" depth="${ct_d*ct_d}" width="${ct_w*ct_w}" height="${ct_h*ct_h}"/>
   </link>
@@ -129,4 +136,5 @@
       <xacro:wheel_dim length="${w_l}" radius="${w_r}"/>
     </collision>
+    <!--length and radius parameters are squared before being passed in, to simplify inertia calculations-->
     <xacro:wheel_inertia mass="${w_m}" length="${w_l*w_l}" radius="${w_r*w_r}" />
   </link>
@@ -138,4 +146,5 @@
       <xacro:wheel_dim length="${w_l}" radius="${w_r}"/>
     </collision>
+    <!--length and radius parameters are squared before being passed in, to simplify inertia calculations-->
     <xacro:wheel_inertia mass="${w_m}" length="${w_l*w_l}" radius="${w_r*w_r}" />
   </link>
@@ -147,4 +156,5 @@
       <xacro:b_dim radius="${b_r}"/>
     </collision>
+    <!--radius parameters are squared before being passed in, to simplify inertia calculations-->
     <xacro:b_inertia mass="${b_m}" radius="${b_r*b_r}"/>
   </link>
@@ -156,10 +166,13 @@
       <xacro:b_dim radius="${b_r}"/>
     </collision>
+    <!--radius parameters are squared before being passed in, to simplify inertia calculations-->
     <xacro:b_inertia mass="${b_m}" radius="${b_r*b_r}"/>
   </link>
+  <!--joint definitions-->
   <joint name = "wb_lw_joint" type = "continuous">
     <parent link = "wheel_base"/>
     <child link= "left_wheel"/>
     <axis xyz = "0 0 1"/>
+    <!--xyz parameters set using macros to allow joint position to scale if the constants are changed-->
     <origin rpy="0 1.57075 1.57075" xyz="0 ${(wb_w/2)+(w_l/2)} 0"/>
     <dynamics friction="14.595"/>
@@ -170,4 +183,5 @@
     <child link= "right_wheel"/>
     <axis xyz = "0 0 1"/>
+    <!--xyz parameters set using macros to allow joint position to scale if the constants are changed-->
     <origin rpy="0 1.57075 1.57075" xyz="0 -${(wb_w/2)+(w_l/2)} 0"/>
     <dynamics friction="14.595"/>
@@ -177,4 +191,5 @@
     <parent link = "wheel_base"/>
     <child link= "bearing_front"/>
+    <!--xyz parameters set using macros to allow joint position to scale if the constants are changed-->
     <origin rpy="0 0 0" xyz="${(wb_w/2)+(w_l/2)} 0 0"/>
   </joint>
@@ -182,4 +197,5 @@
     <parent link = "wheel_base"/>
     <child link= "bearing_rear"/>
+    <!--xyz parameters set using macros to allow joint position to scale if the constants are changed-->
     <origin rpy="0 0 0" xyz="-${(wb_w/2)+(w_l/2)} 0 0"/>
   </joint>
@@ -187,4 +203,5 @@
     <parent link = "wheel_base"/>
     <child link= "support_lf"/>
+    <!--xyz parameters set using macros to allow joint position to scale if the constants are changed-->
     <origin rpy="0 0 0" xyz="${ct_w/1.77/2} ${ct_d/1.77/2} ${(wb_h/2)+(p_l/2)}"/>
   </joint>
@@ -192,4 +209,5 @@
     <parent link = "wheel_base"/>
     <child link= "support_lr"/>
+    <!--xyz parameters set using macros to allow joint position to scale if the constants are changed-->
     <origin rpy="0 0 0" xyz="${ct_w/1.77/2} -${ct_d/1.77/2} ${(wb_h/2)+(p_l/2)}"/>
   </joint>
@@ -197,4 +215,5 @@
     <parent link = "wheel_base"/>
     <child link= "support_rf"/>
+    <!--xyz parameters set using macros to allow joint position to scale if the constants are changed-->
     <origin rpy="0 0 0" xyz="${-ct_w/1.77/2} ${ct_d/1.77/2} ${(wb_h/2)+(p_l/2)}"/>
   </joint>
@@ -202,4 +221,5 @@
     <parent link = "wheel_base"/>
     <child link= "support_rr"/>
+    <!--xyz parameters set using macros to allow joint position to scale if the constants are changed-->
     <origin rpy="0 0 0" xyz="-${ct_w/1.77/2} -${ct_d/1.77/2} ${(wb_h/2)+(p_l/2)}"/>
   </joint>
@@ -207,4 +227,5 @@
     <parent link = "wheel_base"/>
     <child link= "cam_tier"/>
+    <!--xyz parameters set using macros to allow joint position to scale if the constants are changed-->
     <origin rpy="0 0 0" xyz="0 0 ${wb_h+p_l}"/>
   </joint>
@@ -213,6 +234,8 @@
     <child link="cam"/>
     <axis xyz="0 1 0" />
+    <!--xyz parameters set using macros to allow joint position to scale if the constants are changed-->
     <origin xyz="0 0 ${2*wb_h+p_l+(camera_link/2)}" rpy="0 0 0"/>
   </joint>
+  <!--transmission definitions-->
   <transmission name="trans_left">
 		<type>transmission_interface/SimpleTransmission</type>
@@ -235,4 +258,5 @@
 		</actuator>
 	</transmission>
+  <!--gazebo camera plugin-->
   <gazebo reference="cam">
     <sensor name="camera" type="wideanglecamera">
